File: motocontro_rev_4.sch (EAGLE design)
At the start: 49 parts

Commit message: Added MOSFET heatsink package
Must re-route and arrange. Probably mess around with making the heatsink smaller or putting an actual heatsink package on top of it.
Parts:
- removed GPIO: (no value), con-lsta:FE06-1
- added U$4: JST-PH_5-PIN_HEADER, JST_headers:JST-PH_5-PIN_HEADER
Connections:
- removed net N$47: GPIO.1, U$2.4/CANRX
- net DGND: now also U$4.5; no longer GPIO.6
- net N$42: now also U$4.4; no longer GPIO.5
- net N$43: now also U$4.3; no longer GPIO.4
- net N$44: now also U$4.2; no longer GPIO.3
- net N$45: now also U$4.1; no longer GPIO.2
Other:
- note added: "replace fan connector with anderson powerpole"
- note removed: "connect a couple of GPIO or input headers hanging off"
- note removed: "put some LEDs as GPIOs to the teensy"
- moved on the sheet: HS_FET, LS_FET

Commit message: LETS GO
Parts:
- added C4: 100 u, adafruit:CPOL-USE10-20
- C2: device adafruit:C-US225-113X268 -> adafruit:CPOL-USE10-20
Connections:
- net PGND: now also C2.-, C4.-; no longer C2.2
- net VBUS: now also C2.+, C4.+; no longer C2.1
Other:
- moved on the sheet: HS_FET, LS_FET

Commit message: adds fuse. zener, caps, dsafksdf;
Parts:
- added D1: 1N4728, diode:1N4728
- added F1: FUSEBLANK_5X20MM, fuse:FUSEBLANK_5X20MM
- added R13, R14, R15: 15k, adafruit:R-US_R0805
- C1: value 1u -> 22u
- C2, C4: value 100 u -> 1000u
Connections:
- new net CLAMPED: C2.+, D1.C, R13.2, R14.2, R15.2, U$3.VI+
- new net FUSED: F1.2, R13.1, R14.1, R15.1
- net PGND: now also D1.A
- net VBUS: now also F1.1; no longer C2.+, U$3.VI+
Other:
- note added: "series resistor from 48V and Zener"
- note removed: "replace fan connector with anderson powerpole"
- moved on the sheet: C2, C4

Commit message: moves stuff around
Parts:
- renumbered SV1 to PGND, SV2 to DGND
Changed lines of the file:
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@@
 <part name="TP8" library="testpad" library_urn="urn:adsk.eagle:library:385" deviceset="PTR1" device="B1,27" package3d_urn="urn:adsk.eagle:package:27944/1"/>
 <part name="OP+" library="testpad" library_urn="urn:adsk.eagle:library:385" deviceset="PTR1" device="B1,27" package3d_urn="urn:adsk.eagle:package:27944/1"/>
-<part name="SV2" library="con-lstb" library_urn="urn:adsk.eagle:library:162" deviceset="MA03-1" device="" package3d_urn="urn:adsk.eagle:package:8339/1"/>
-<part name="SV1" library="con-lstb" library_urn="urn:adsk.eagle:library:162" deviceset="MA03-1" device="" package3d_urn="urn:adsk.eagle:package:8339/1"/>
+<part name="DGND" library="con-lstb" library_urn="urn:adsk.eagle:library:162" deviceset="MA03-1" device="" package3d_urn="urn:adsk.eagle:package:8339/1"/>
+<part name="PGND" library="con-lstb" library_urn="urn:adsk.eagle:library:162" deviceset="MA03-1" device="" package3d_urn="urn:adsk.eagle:package:8339/1"/>
 <part name="STATUS" library="adafruit" library_urn="urn:adsk.eagle:library:420" deviceset="LED" device="CHIP-LED0805"/>
 <part name="R12" library="adafruit" library_urn="urn:adsk.eagle:library:420" deviceset="R-US_" device="R0805" value="150"/>
@@
 <attribute name="TP_SIGNAL_NAME" x="24.13" y="-27.94" size="1.778" layer="97" rot="R180"/>
 </instance>
-<instance part="SV2" gate="G$1" x="-160.02" y="-63.5" smashed="yes" rot="R180">
+<instance part="DGND" gate="G$1" x="-160.02" y="-63.5" smashed="yes" rot="R180">
 <attribute name="VALUE" x="-158.75" y="-55.88" size="1.778" layer="96" rot="R180"/>
 <attribute name="NAME" x="-158.75" y="-69.342" size="1.778" layer="95" rot="R180"/>
 </instance>
-<instance part="SV1" gate="G$1" x="-160.02" y="-78.74" smashed="yes" rot="R180">
+<instance part="PGND" gate="G$1" x="-160.02" y="-78.74" smashed="yes" rot="R180">
 <attribute name="VALUE" x="-158.75" y="-71.12" size="1.778" layer="96" rot="R180"/>
 <attribute name="NAME" x="-158.75" y="-84.582" size="1.778" layer="95" rot="R180"/>
@@
 <label x="-185.42" y="-76.2" size="1.778" layer="95"/>
 <pinref part="R11" gate="G$1" pin="1"/>
-<pinref part="SV1" gate="G$1" pin="1"/>
+<pinref part="PGND" gate="G$1" pin="1"/>
 <wire x1="-167.64" y1="-76.2" x2="-180.34" y2="-76.2" width="0.1524" layer="91"/>
-<pinref part="SV1" gate="G$1" pin="2"/>
+<pinref part="PGND" gate="G$1" pin="2"/>
 <wire x1="-167.64" y1="-78.74" x2="-180.34" y2="-78.74" width="0.1524" layer="91"/>
 <wire x1="-180.34" y1="-78.74" x2="-180.34" y2="-76.2" width="0.1524" layer="91"/>
 <junction x="-180.34" y="-76.2"/>
-<pinref part="SV1" gate="G$1" pin="3"/>
+<pinref part="PGND" gate="G$1" pin="3"/>
 <wire x1="-167.64" y1="-81.28" x2="-180.34" y2="-81.28" width="0.1524" layer="91"/>
 <wire x1="-180.34" y1="-81.28" x2="-180.34" y2="-78.74" width="0.1524" layer="91"/>
@@
 <label x="-185.42" y="-66.04" size="1.778" layer="95"/>
 <pinref part="R11" gate="G$1" pin="2"/>
-<pinref part="SV2" gate="G$1" pin="1"/>
+<pinref part="DGND" gate="G$1" pin="1"/>
 <wire x1="-167.64" y1="-60.96" x2="-180.34" y2="-60.96" width="0.1524" layer="91"/>
 <wire x1="-180.34" y1="-60.96" x2="-180.34" y2="-63.5" width="0.1524" layer="91"/>
-<pinref part="SV2" gate="G$1" pin="2"/>
+<pinref part="DGND" gate="G$1" pin="2"/>
 <wire x1="-180.34" y1="-63.5" x2="-180.34" y2="-66.04" width="0.1524" layer="91"/>
 <wire x1="-167.64" y1="-63.5" x2="-180.34" y2="-63.5" width="0.1524" layer="91"/>
 <junction x="-180.34" y="-63.5"/>
-<pinref part="SV2" gate="G$1" pin="3"/>
+<pinref part="DGND" gate="G$1" pin="3"/>
 <wire x1="-167.64" y1="-66.04" x2="-180.34" y2="-66.04" width="0.1524" layer="91"/>
 <junction x="-180.34" y="-66.04"/>

Commit message: makes edits for resping
Parts:
- removed PWM: PTR1B1,27, testpad:PTR1B1,27
- removed R13, R14, R15: 15k, adafruit:R-US_R0805
- added TP1: PTR2, testpad:PTR2
- added U$5: 8-PIN-MOLEX-RA-FEMALE, master_library:8-PIN-MOLEX-RA-FEMALE
- BATTERY: device motor controller rev 3.0.6:BATTERY -> Rev_motor_controller_3.02:BATTERY
- C2: device adafruit:CPOL-USE10-20 -> adafruit:CPOL-USE5-13
- CSD: value (none) -> 47 pF
- MOTOR: device motor controller rev 3.0.6:MOTOR -> Rev_motor_controller_3.02:MOTOR
- R10, R12, R8: value 150 -> 300
- R2: value 7k -> 10k
- R3, R4: value (none) -> 0
- R9: value 150 -> 1k
- RSD: value (none) -> 10k
- U$1: value L6390_DRIVER -> L6390SO-16NARRROW; device motocontro_rev_4:L6390_DRIVER -> master_library:L6390SO-16NARRROW
- U$4: value JST-PH_5-PIN_HEADER -> 8-PIN-MOLEX-RA-FEMALE; device JST_headers:JST-PH_5-PIN_HEADER -> master_library:8-PIN-MOLEX-RA-FEMALE
Connections:
- net FAULT_LED renamed OCP_OUT
- net VBUS renamed HVBUS
- removed net FUSED: F1.2, R13.1, R14.1, R15.1
- removed net N$42: U$2.0/RX, U$4.4
- removed net N$43: U$2.1/TX, U$4.3
- removed net N$44: U$2.2, U$4.2
- removed net N$45: U$2.3/CANTX, U$4.1
- removed net PWM: PWM.TP, U$1.1_LIN, U$1.3_HIN, U$2.30
- new net /LIN: TP1-1.TP, U$1.1_LIN, U$2.30
- new net BRAKE: U$2.2, U$4.P$1
- new net CURRENT_IN: OPOUT.TP, U$2.14/A0
- new net ENCXA: U$2.3/CANTX, U$5.P$2
- new net ENCXB: U$2.4/CANRX, U$5.P$3
- new net ENCYA: U$2.32/A13, U$5.P$6
- new net ENCYB: U$2.25, U$5.P$7
- new net GPIO0: U$2.0/RX, U$4.P$7
- new net GPIO1: U$2.1/TX, U$4.P$6
- new net HIN: TP1-2.TP, U$1.3_HIN, U$2.29
- new net OCP_IN: SD.TP, U$2.24
- new net PEDAL_IN: U$2.16/A2, U$4.P$2
- net 5V: now also RSD.2, U$5.P$1, U$5.P$5
- net CLAMPED: now also F1.2; no longer R13.2, R14.2, R15.2
- net DGND: now also U$4.P$8, U$5.P$4, U$5.P$8; no longer U$4.5
- net N$4: now also U$2.31/A12; no longer U$2.32/A13
- net OPOUT: no longer OPOUT.TP, U$2.14/A0
- net SD/OD: no longer SD.TP, U$2.24
- net VCC: no longer RSD.2
Other:
- note removed: "Make an SPI bus to run to an OLED display in the front"
- moved on the sheet: C2, C3, C4, DGND, F1, FAN, LED1, LED2, LED3, OPOUT, PGND, R10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

Commit message: fixes merge issues
Other:
- note added: "change the package for this part (thinner)"
Changed lines of the file:
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@@
 <text x="124.46" y="-11.176" size="1.778" layer="94">consider adding two in parallel </text>
 <text x="-274.32" y="35.56" size="1.778" layer="91">series resistor from 48V and Zener</text>
+<text x="-236.22" y="35.56" size="1.778" layer="91">series resistor from 48V and Zener</text>
+<text x="0" y="48.26" size="1.778" layer="91">change the package for this part (thinner) </text>
 </plain>
 <instances>
