File: motocontro_rev_4.brd (EAGLE design)
At the start: 163 x 89 mm, 50 parts

Commit message: adds fuse. zener, caps, dsafksdf;
Parts:
- added D1: 1N4728, diode:DO41Z10
- added F1: FUSEBLANK_5X20MM, fuse:FUSE_HOLDER_5X20MM
- added R13, R14, R15: 15k, adafruit:R0805
- C1: value 1u -> 22u
- C2, C4: value 100 u -> 1000u
- moved C2 50.0 mm to (29.3, 5.81)
- moved HS_FET 8.51 mm to (104.6, 65.9), turned to 0 degrees
- moved OP+ 6.40 mm to (76.5, 37.0)
- moved HVG 4.72 mm to (84.0, 64.5)
- moved R5 4.00 mm to (78.8, 44.3)
- moved BATTERY 3.50 mm to (116.5, 5.08)
- moved R6 3.00 mm to (75.9, 46.9)
- moved R7 3.00 mm to (75.8, 41.9)
Connections:
- new net CLAMPED: C2.+, D1.C, R13.2, R14.2, R15.2, U$3.VI+
- new net FUSED: F1.2, R13.1, R14.1, R15.1
- net PGND: now also D1.A
- net VBUS: now also F1.1; no longer C2.+, U$3.VI+
Routing:
- net OUT: track 28.0 -> 47.7 mm
- net VBUS: track 17.0 -> 13.4 mm
- net OP+: track 19.6 -> 20.8 mm
- net RSENSE+: track 32.6 -> 33.8 mm
- net CLAMPED: track 0.00 -> 0.57 mm
- added copper zone on layer 16, net CLAMPED
- added copper zone on layer 16, net FUSED
Other:
- board text added: "add fuse holder"

Commit message: moves stuff around
Parts:
- moved C2 2.69 mm to (30.3, 8.31)
- renumbered SV1 to PGND, SV2 to DGND
Routing:
- net CLAMPED: track 0.57 -> 0.00 mm
- net DGND: track 55.2 -> 55.7 mm
- net OUT: vias 98 -> 102
Other:
- board text added: "Custom Built for SEM by M&M. LET'S GO rrrrriiiIIICE"
- board text added: "REVolution MC 2018.1"
- board text removed: "Custom Built for SEM by M&M LETS GO RICE"
- board text removed: "REV MC 2018.1"
- board text removed: "add fuse holder"
Changed lines of the file:
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@@
 <wire x1="163" y1="89" x2="0" y2="89" width="0" layer="20"/>
 <wire x1="0" y1="89" x2="0" y2="0" width="0" layer="20"/>
-<text x="11" y="83" size="2.54" layer="25">REV MC 2018.1</text>
+<text x="11" y="83" size="2.54" layer="25">REVolution MC 2018.1</text>
 <dimension x1="160" y1="0" x2="160" y2="89" x3="175.5" y3="44.5" textsize="1.778" layer="20"/>
-<hole x="4.5" y="85" drill="2"/>
-<hole x="4.5" y="85" drill="2"/>
+<hole x="4" y="85" drill="2"/>
 <hole x="4.5" y="4" drill="2"/>
 <hole x="158.5" y="4" drill="2"/>
@@
 </polygon>
 <polygon width="0.4064" layer="30">
-<vertex x="96.5" y="53.5"/>
-<vertex x="96.5" y="32"/>
+<vertex x="97" y="53.5"/>
+<vertex x="97" y="31.5"/>
 <vertex x="97.5" y="31"/>
 <vertex x="130.5" y="31"/>
@@
 <vertex x="151" y="83"/>
 </polygon>
-<text x="82" y="83" size="1.778" layer="21">Custom Built for SEM by M&amp;M
-LETS GO RICE</text>
+<text x="72.5" y="80" size="1.778" layer="21">Custom Built for SEM by M&amp;M.
+LET'S GO rrrrriiiIIICE
+</text>
 <dimension x1="0" y1="89" x2="163" y2="89" x3="81.5" y3="93" textsize="1.778" layer="20" dtype="horizontal"/>
-<text x="10.5" y="90" size="1.778" layer="27">add fuse holder</text>
 </plain>
 <attributes>
@@
 <element name="LDO" library="r-78xx_10" package="SIP3" value="TRACO-TSR-1-2450" x="68.95" y="27.17" smashed="yes" rot="R270">
 <attribute name="NAME" x="74.9" y="32.87" size="1.27" layer="25" rot="R270"/>
-<attribute name="VALUE" x="65.25" y="32.87" size="1.27" layer="27" rot="R270"/>
 </element>
 <element name="C3" library="adafruit" library_urn="urn:adsk.eagle:library:420" package="153CLV-0605" value="22u" x="60.62" y="26.44" smashed="yes" rot="R90">
@@
 <attribute name="VALUE" x="56.43" y="55.51" size="1.27" layer="27" rot="R270"/>
 </element>
-<element name="C2" library="adafruit" library_urn="urn:adsk.eagle:library:420" package="EB20D" value="1000u" x="29.31" y="5.81" smashed="yes">
-<attribute name="NAME" x="16.356" y="11.779" size="1.778" layer="25" ratio="10"/>
-<attribute name="VALUE" x="24.23" y="3.27" size="1.778" layer="27" ratio="10"/>
+<element name="C2" library="adafruit" library_urn="urn:adsk.eagle:library:420" package="EB20D" value="1000u" x="30.31" y="8.31" smashed="yes">
+<attribute name="NAME" x="17.356" y="14.279" size="1.778" layer="25" ratio="10"/>
+<attribute name="VALUE" x="25.23" y="5.77" size="1.778" layer="27" ratio="10"/>
 </element>
 <element name="R5" library="adafruit" library_urn="urn:adsk.eagle:library:420" package="R0805" value="1k" x="78.839" y="44.253" smashed="yes">
@@
 <attribute name="VALUE" x="75.865" y="36.238" size="0.0254" layer="27"/>
 </element>
-<element name="SV2" library="con-lstb" library_urn="urn:adsk.eagle:library:162" package="MA03-1" package3d_urn="urn:adsk.eagle:package:8339/1" value="" x="74.5" y="74.5" smashed="yes" rot="R270">
+<element name="DGND" library="con-lstb" library_urn="urn:adsk.eagle:library:162" package="MA03-1" package3d_urn="urn:adsk.eagle:package:8339/1" value="" x="74.5" y="74.5" smashed="yes" rot="R270">
 <attribute name="MF" value="" x="74.5" y="74.5" size="1.778" layer="27" rot="R270" display="off"/>
 <attribute name="MPN" value="" x="74.5" y="74.5" size="1.778" layer="27" rot="R270" display="off"/>
@@
 <attribute name="VALUE" x="71.579" y="78.31" size="1.27" layer="27" ratio="10" rot="R270"/>
 </element>
-<element name="SV1" library="con-lstb" library_urn="urn:adsk.eagle:library:162" package="MA03-1" package3d_urn="urn:adsk.eagle:package:8339/1" value="" x="87.5" y="19.5" smashed="yes">
+<element name="PGND" library="con-lstb" library_urn="urn:adsk.eagle:library:162" package="MA03-1" package3d_urn="urn:adsk.eagle:package:8339/1" value="" x="87.5" y="19.5" smashed="yes">
 <attribute name="MF" value="" x="87.5" y="19.5" size="1.778" layer="27" display="off"/>
 <attribute name="MPN" value="" x="87.5" y="19.5" size="1.778" layer="27" display="off"/>
@@
 <attribute name="OC_FARNELL" value="unknown" x="82" y="8" size="1.778" layer="27" rot="R180" display="off"/>
 <attribute name="OC_NEWARK" value="unknown" x="82" y="8" size="1.778" layer="27" rot="R180" display="off"/>
-<attribute name="VALUE" x="86.4196" y="13.461" size="1.778" layer="27" ratio="10" rot="R180"/>
 </element>
 </elements>
@@
 <wire x1="89.5" y1="59.5" x2="89.5" y2="58.5" width="0.6096" layer="16"/>
 <via x="89.5" y="58.5" extent="1-16" drill="0.35"/>
+<via x="107.5" y="44.5" extent="1-16" drill="0.35"/>
+<via x="109" y="44.5" extent="1-16" drill="0.35"/>
+<via x="109" y="49" extent="1-16" drill="0.35"/>
+<via x="107.5" y="49" extent="1-16" drill="0.35"/>
 </signal>
 <signal name="VBUS">
@@
 <wire x1="67" y1="43" x2="74" y2="36" width="0.4064" layer="16"/>
 <contactref element="R11" pad="1"/>
-<contactref element="SV1" pad="1"/>
-<contactref element="SV1" pad="2"/>
-<contactref element="SV1" pad="3"/>
+<contactref element="PGND" pad="1"/>
+<contactref element="PGND" pad="2"/>
+<contactref element="PGND" pad="3"/>
 <polygon width="1.016" layer="1">
 <vertex x="1.5" y="23.5"/>
@@
 <contactref element="R10" pad="1"/>
 <contactref element="R11" pad="2"/>
-<contactref element="SV2" pad="1"/>
-<contactref element="SV2" pad="2"/>
-<contactref element="SV2" pad="3"/>
+<contactref element="DGND" pad="1"/>
+<contactref element="DGND" pad="2"/>
+<contactref element="DGND" pad="3"/>
 <wire x1="60.62" y1="23.74" x2="59.14" y2="22.26" width="0.6096" layer="1"/>
 <wire x1="59.14" y1="22.26" x2="47.61" y2="22.26" width="0.6096" layer="1"/>
-<via x="69.5" y="20" extent="1-16" drill="0.35"/>
 <wire x1="21" y1="79.5" x2="23.54" y2="79.5" width="0.8128" layer="16"/>
 <wire x1="23.54" y1="79.5" x2="26.5" y2="76.54" width="0.8128" layer="16"/>
@@
 <vertex x="28.5" y="75.5"/>
 </polygon>
-<wire x1="70" y1="17.5" x2="70" y2="19.5" width="0.6096" layer="1"/>
-<wire x1="70" y1="19.5" x2="69.5" y2="20" width="0.6096" layer="1"/>
+<via x="69.5" y="20.5" extent="1-16" drill="0.35"/>
+<wire x1="70" y1="20" x2="69.5" y2="20.5" width="1.016" layer="1"/>
+<wire x1="70" y1="17.5" x2="70" y2="20" width="1.016" layer="1"/>
 </signal>
 <signal name="OPOUT">
@@
 <contactref element="R13" pad="2"/>
 <contactref element="R14" pad="2"/>
-<wire x1="5.54" y1="21.46" x2="6.11" y2="21.46" width="0.2" layer="1"/>
 <contactref element="C2" pad="+"/>
 <polygon width="0.6096" layer="16">

Commit message: makes edits for resping
Parts:
- removed PWM: PTR1B1,27, testpad:B1,27
- removed R13, R14, R15: 15k, adafruit:R0805
- added TP1: PTR2, testpad:P2-38-17
- added U$5: 8-PIN-MOLEX-RA-FEMALE, master_library:8-PIN-MOLEX
- BATTERY, MOTOR: device motor controller rev 3.0.6:SB50POWER_CLAW -> Rev_motor_controller_3.02:SB50POWER_CLAW
- C2: device adafruit:EB20D -> adafruit:E5-13
- CSD: value (none) -> 47 pF
- R10, R12, R8: value 150 -> 300
- R2: value 7k -> 10k
- R3, R4: value (none) -> 0
- R9: value 150 -> 1k
- RSD: value (none) -> 10k
- U$1: value L6390_DRIVER -> L6390SO-16NARRROW; device motocontro_rev_4:SOIC127P1032X265-16 -> master_library:SO-16NARROW
- U$4: value JST-PH_5-PIN_HEADER -> 8-PIN-MOLEX-RA-FEMALE; device JST_headers:JST_B5B-PH_HEADER -> master_library:8-PIN-MOLEX
- moved U$4 83.6 mm to (0.50, -36.0), turned to 0 degrees
- moved C2 6.52 mm to (23.8, 8.81)
- moved U$1 5.39 mm to (69.1, 61.7), turned to 270 degrees
Connections:
- net FAULT_LED renamed OCP_OUT
- net VBUS renamed HVBUS
- removed net FUSED: F1.2, R13.1, R14.1, R15.1
- removed net N$42: U$2.0/RX, U$4.P4
- removed net N$43: U$2.1/TX, U$4.P3
- removed net N$44: U$2.2, U$4.P2
- removed net N$45: U$2.3/CANTX, U$4.P1
- removed net PWM: PWM.TP, U$1.1, U$1.3, U$2.30
- new net /LIN: TP1.TP-1, U$1.P$1, U$2.30
- new net BRAKE: U$2.2, U$4.P1
- new net CURRENT_IN: OPOUT.TP, U$2.14/A0
- new net ENCXA: U$2.3/CANTX, U$5.P2
- new net ENCXB: U$2.4/CANRX, U$5.P3
- new net ENCYA: U$2.32/A13, U$5.P6
- new net ENCYB: U$2.25, U$5.P7
- new net GPIO0: U$2.0/RX, U$4.P7
- new net GPIO1: U$2.1/TX, U$4.P6
- new net HIN: TP1.TP-2, U$1.P$3, U$2.29
- new net OCP_IN: SD.TP, U$2.24
- new net PEDAL_IN: U$2.16/A2, U$4.P2
- net 5V: now also RSD.2, U$5.P1, U$5.P5
- net CLAMPED: now also F1.2; no longer R13.2, R14.2, R15.2
- net DGND: now also U$1.P$8, U$4.P8, U$5.P4, U$5.P8; no longer U$1.8, U$4.P5
- net DT: now also U$1.P$5; no longer U$1.5
- net HVG: now also U$1.P$10; no longer U$1.15
- net LVG: now also U$1.P$14; no longer U$1.11
- net N$4: now also U$2.31/A12; no longer U$2.32/A13
- net OP+: now also U$1.P$16; no longer U$1.9
- net OP-: now also U$1.P$6; no longer U$1.6
- net OPOUT: now also U$1.P$7; no longer OPOUT.TP, U$1.7, U$2.14/A0
- net OUT: now also U$1.P$11; no longer U$1.14
- net RSENSE+: now also U$1.P$15; no longer U$1.10
- net SD/OD: now also U$1.P$2; no longer SD.TP, U$1.2, U$2.24
- net VBOOT: now also U$1.P$9; no longer U$1.16
- net VCC: now also U$1.P$4; no longer RSD.2, U$1.4
Routing:
- net /LIN: track 0.00 -> 45.3 mm, vias 0 -> 2
- net PWM: track 34.7 -> 0.00 mm, vias 2 -> 0
- net OPOUT: track 50.1 -> 40.5 mm
- net N$42: track 6.25 -> 0.00 mm
- net OP-: track 16.8 -> 22.9 mm
- net N$43: track 6.03 -> 0.00 mm
- net DT: track 16.5 -> 22.5 mm
- net DGND: track 55.7 -> 61.7 mm, vias 7 -> 6
- net N$44: track 5.81 -> 0.00 mm
- net N$45: track 5.58 -> 0.00 mm
- net VBOOT: track 9.17 -> 13.6 mm
- net N$4: track 4.47 -> 0.00 mm
- net RSENSE+: track 33.8 -> 37.0 mm
- net SD/OD: track 26.3 -> 29.0 mm
- net OP+: track 20.8 -> 23.3 mm
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